File: kicad/linkpodule.kicad_sch (KiCad schematic)
At the start: 25 parts, among them IC1 74HCT245, IC2 74HCT245, IC3 N82S123AN, IC4 PAL16L8-25, IC5A1 IMSC011, IC5B1 IMSC012, IC6 5MHZ, IC7 74HCT175, IC8 74HCT244, J1 DIN41612_02x32_AC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

Commit message: kicad: Add missing D3 connection on PAL
Connections:
- net B_BD3: now also IC4.19 (~{O_{8}})
Changed lines of the file:
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@@
 	(wire
 		(pts
-			(xy 196.85 82.55) (xy 208.28 82.55)
+			(xy 196.85 82.55) (xy 209.55 82.55)
 		)
 		(stroke
@@
 	(wire
 		(pts
+			(xy 196.85 85.09) (xy 209.55 85.09)
+		)
+		(stroke
+			(width 0)
+			(type default)
+		)
+	)
+	(wire
+		(pts
 			(xy 259.08 45.72) (xy 259.08 93.98)
 		)
@@
 		(effects
 			(font
+				(size 1.27 1.27)
+			)
+			(justify left bottom)
+		)
+	)
+	(label "B_BD3"
+		(at 199.39 85.09 0)
+		(effects
+			(font
